File: keyboard-pcb-proj-best/keyboard-pcb-proj-best.kicad_pcb (KiCad board)
At the start: 2 copper layers, 76.2 x 38.1 mm, 24 parts, among them SW1 SW_PUSH, U1 ATmega32U4-A, Y1 16Mhz

Commit message: Fixed Most Errors
Parts:
- moved USB1 0.79 mm to (175.1, 36.0)
Routing:
- net unconnected-(USB1-SHIELD-Pad6): track 0.00 -> 16.3 mm
- net VCC: track 13.3 -> 12.5 mm
- net D-: track 6.64 -> 5.84 mm
- net D+: track 6.48 -> 5.69 mm
- net GND: track 127.2 -> 126.4 mm
Changed lines of the file:
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@@
 	(footprint "random-keyboard-parts:Molex-0548190589"
 		(layer "B.Cu")
-		(at 175.1 35.1875 -90)
+		(at 175.1 35.98125 -90)
 		(property "Reference" "USB1"
-			(at 2.032 0 0)
+			(at 2.032 0 180)
 			(layer "B.SilkS")
 			(effects
@@
 		)
 		(property "Value" "Molex-0548190589"
-			(at -5.08 0 0)
+			(at -5.08 0 180)
 			(layer "Dwgs.User")
 			(effects
@@
 		(attr smd)
 		(fp_line
-			(start 0 3.85)
-			(end 5.45 3.85)
-			(stroke
-				(width 0.15)
-				(type solid)
-			)
-			(layer "B.SilkS")
-		)
-		(fp_line
-			(start 5.45 3.85)
-			(end 5.45 -3.85)
-			(stroke
-				(width 0.15)
-				(type solid)
-			)
-			(layer "B.SilkS")
-		)
-		(fp_line
-			(start 0 -3.85)
-			(end 5.45 -3.85)
-			(stroke
-				(width 0.15)
-				(type solid)
-			)
-			(layer "B.SilkS")
-		)
-		(fp_line
 			(start -1.75 4.572)
 			(end -1.75 -4.572)
@@
 		(fp_line
 			(start -3.75 3.85)
-			(end 0 3.85)
-			(stroke
-				(width 0.15)
-				(type solid)
-			)
-			(layer "Dwgs.User")
-		)
-		(fp_line
-			(start -3.75 3.85)
 			(end -3.75 -3.85)
 			(stroke
@@
 		)
 		(fp_line
-			(start -3.75 -3.85)
-			(end 0 -3.85)
-			(stroke
-				(width 0.15)
-				(type solid)
-			)
-			(layer "Dwgs.User")
-		)
-		(fp_line
 			(start -3.75 3.75)
 			(end 5.5 3.75)
@@
 		)
 		(fp_line
-			(start 3.25 2)
-			(end 3.25 -2)
+			(start 5.5 2)
+			(end 5.5 -2)
 			(stroke
-				(width 0.15)
-				(type solid)
+				(width 0.05)
+				(type default)
 			)
 			(layer "B.CrtYd")
 		)
 		(fp_line
-			(start 5.5 2)
-			(end 3.25 2)
+			(start -3.75 -3.75)
+			(end -3.75 3.75)
 			(stroke
 				(width 0.15)
@@
 		)
 		(fp_line
-			(start 3.25 1.25)
-			(end 5.5 1.25)
+			(start 5.5 -3.75)
+			(end -3.75 -3.75)
 			(stroke
 				(width 0.15)
@@
 			(layer "B.CrtYd")
 		)
-		(fp_line
-			(start 5.5 0.5)
-			(end 3.25 0.5)
+		(fp_rect
+			(start 3.25 2)
+			(end 5.5 -1.25)
 			(stroke
 				(width 0.15)
 				(type solid)
 			)
+			(fill no)
 			(layer "B.CrtYd")
 		)
-		(fp_line
-			(start 3.25 -0.5)
-			(end 5.5 -0.5)
+		(fp_rect
+			(start 5.5 2)
+			(end 5.5 1.25)
 			(stroke
-				(width 0.15)
-				(type solid)
+				(width 0.05)
+				(type default)
 			)
+			(fill no)
 			(layer "B.CrtYd")
 		)
-		(fp_line
-			(start 5.5 -1.25)
-			(end 3.25 -1.25)
+		(fp_rect
+			(start 3.25 1.25)
+			(end 5.5 0.5)
 			(stroke
 				(width 0.15)
 				(type solid)
 			)
+			(fill no)
 			(layer "B.CrtYd")
 		)
-		(fp_line
-			(start 3.25 -2)
-			(end 5.5 -2)
+		(fp_rect
+			(start 3.25 0.5)
+			(end 5.5 -0.5)
 			(stroke
 				(width 0.15)
 				(type solid)
 			)
+			(fill no)
 			(layer "B.CrtYd")
 		)
-		(fp_line
-			(start -3.75 -3.75)
-			(end -3.75 3.75)
+		(fp_rect
+			(start 3.25 -0.5)
+			(end 5.5 -1.25)
 			(stroke
 				(width 0.15)
 				(type solid)
 			)
+			(fill no)
 			(layer "B.CrtYd")
 		)
-		(fp_line
-			(start 5.5 -3.75)
-			(end -3.75 -3.75)
+		(fp_rect
+			(start 3.25 -1.25)
+			(end 5.5 -2)
 			(stroke
 				(width 0.15)
 				(type solid)
 			)
+			(fill no)
 			(layer "B.CrtYd")
 		)
 		(fp_text user "${REFERENCE}"
-			(at 2 0 0)
+			(at 2 0 180)
 			(layer "B.CrtYd")
 			(effects
@@
 		(layer "Edge.Cuts")
 	)
+	(gr_line
+		(start 173.85 41.48125)
+		(end 173.85 39.23125)
+		(stroke
+			(width 0.05)
+			(type default)
+		)
+		(layer "B.CrtYd")
+	)
+	(gr_line
+		(start 175.6 41.48125)
+		(end 175.6 39.23125)
+		(stroke
+			(width 0.05)
+			(type default)
+		)
+		(layer "B.CrtYd")
+	)
+	(gr_rect
+		(start 173.1 39.23125)
+		(end 177.1 41.48125)
+		(stroke
+			(width 0.05)
+			(type default)
+		)
+		(fill no)
+		(layer "B.CrtYd")
+	)
+	(gr_line
+		(start 176.35 39.23125)
+		(end 176.35 41.48125)
+		(stroke
+			(width 0.05)
+			(type default)
+		)
+		(layer "B.CrtYd")
+	)
+	(gr_line
+		(start 174.6 39.23125)
+		(end 174.6 41.48125)
+		(stroke
+			(width 0.05)
+			(type default)
+		)
+		(layer "B.CrtYd")
+	)
+	(gr_line
+		(start 175.6 39.23125)
+		(end 176.35 39.23125)
+		(stroke
+			(width 0.05)
+			(type default)
+		)
+		(layer "B.CrtYd")
+	)
+	(gr_line
+		(start 173.1 41.48125)
+		(end 173.1 39.23125)
+		(stroke
+			(width 0.05)
+			(type default)
+		)
+		(layer "B.CrtYd")
+	)
+	(gr_line
+		(start 176.35 39.23125)
+		(end 176.35 41.48125)
+		(stroke
+			(width 0.05)
+			(type default)
+		)
+		(layer "B.CrtYd")
+	)
+	(gr_line
+		(start 177.1 39.23125)
+		(end 176.35 39.23125)
+		(stroke
+			(width 0.05)
+			(type default)
+		)
+		(layer "B.CrtYd")
+	)
 	(segment
 		(start 184.6375 50.8)
@@
 	)
 	(segment
-		(start 184.95 42.86875)
-		(end 184.95 44.06875)
-		(width 0.3556)
-		(layer "B.Cu")
-		(net 2)
-	)
-	(segment
 		(start 196.88125 54.8)
 		(end 196.88125 58.15625)
@@
 	)
 	(segment
+		(start 177.81875 42.475)
+		(end 183.35625 42.475)
+		(width 0.3556)
+		(layer "B.Cu")
+		(net 2)
+	)
+	(segment
 		(start 187.21875 41.38125)
 		(end 189.7125 41.38125)
@@
 	)
 	(segment
+		(start 183.35625 42.475)
+		(end 184.95 44.06875)
+		(width 0.3556)
+		(layer "B.Cu")
+		(net 2)
+	)
+	(segment
 		(start 182.5625 52.3875)
 		(end 183.46875 53.29375)
@@
 	)
 	(segment
+		(start 176.7 41.35625)
+		(end 177.81875 42.475)
+		(width 0.3556)
+		(layer "B.Cu")
+		(net 2)
+	)
+	(segment
 		(start 198.606251 48.49375)
 		(end 199.34375 48.49375)
@@
 	)
 	(segment
-		(start 178.59375 42.06875)
-		(end 176.7 40.175)
-		(width 0.3556)
-		(layer "B.Cu")
-		(net 2)
-	)
-	(segment
 		(start 198.4375 65.0875)
 		(end 197.1625 63.8125)
@@
 	)
 	(segment
-		(start 178.59375 42.06875)
-		(end 184.94375 42.06875)
-		(width 0.3556)
-		(layer "B.Cu")
-		(net 2)
-	)
-	(segment
 		(start 189.21875 61.60625)
 		(end 190.5 60.325)
@@
 	)
 	(segment
-		(start 184.94375 42.06875)
-		(end 184.94375 42.8625)
+		(start 176.7 40.48125)
+		(end 176.7 41.35625)
 		(width 0.3556)
 		(layer "B.Cu")
@@
 	)
 	(segment
-		(start 184.94375 42.8625)
-		(end 184.95 42.86875)
-		(width 0.3556)
-		(layer "B.Cu")
-		(net 2)
-	)
-	(segment
 		(start 197.1625 63.8125)
 		(end 197.1625 62.01875)
@@
 	)
 	(segment
-		(start 173.0375 42.8625)
+		(start 173.5 40.48125)
 		(end 173.5 42.4)
 		(width 0.3556)
@@
 	)
 	(segment
-		(start 173.5 42.4)
-		(end 173.5 39.6875)
+		(start 173.0375 42.8625)
+		(end 173.5 42.4)
 		(width 0.3556)
 		(layer "B.Cu")
@@
 	)
 	(segment
-		(start 175.1 44.9125)
-		(end 175.1 39.6875)
+		(start 175.1 40.48125)
+		(end 175.1 44.9125)
 		(width 0.2)
 		(layer "B.Cu")
@@
 	)
 	(segment
-		(start 174.3 44.5375)
-		(end 174.3 39.6875)
+		(start 174.3 40.48125)
+		(end 174.3 44.5375)
 		(width 0.2)
 		(layer "B.Cu")
@@
 		(net 20)
 	)
+	(segment
+		(start 171.45 39.6875)
+		(end 171.45 35.1875)
+		(width 0.254)
+		(layer "B.Cu")
+		(net 43)
+	)
+	(segment
+		(start 171.45 35.1875)
+		(end 178.75 35.1875)
+		(width 0.254)
+		(layer "B.Cu")
+		(net 43)
+	)
+	(segment
+		(start 178.75 35.1875)
+		(end 178.75 39.6875)
+		(width 0.254)
+		(layer "B.Cu")
+		(net 43)
+	)
 	(zone
 		(net 2)
@@
 			)
 		)
+	)
+	(zone
+		(net 2)
+		(net_name "GND")
+		(layer "B.Cu")
+		(hatch edge 0.5)
+		(priority 1)
+		(connect_pads
+			(clearance 0.5)
+		)
+		(min_thickness 0.25)
+		(filled_areas_thickness no)
+		(fill yes
+			(thermal_gap 0.5)
+			(thermal_bridge_width 0.5)
+		)
+		(polygon
+			(pts
+				(xy 167.48125 33.3375) (xy 205.58125 33.3375) (xy 205.58125 71.4375) (xy 167.48125 71.4375)
+			)
+		)
